File: Unified-Daughterboard.kicad_pcb (KiCad board)
At the start: 2 copper layers, 44.7 x 8.7 mm, 9 parts, among them J1 HRO-TYPE-C-31-M-12, J2 Conn_01x04

Commit message: update dboard
Parts:
- removed C1: 4.7n, Capacitor_SMD:C_0603_1608Metric
- removed J1: HRO-TYPE-C-31-M-12, Type-C:HRO-TYPE-C-31-M-12-jlc
- removed R3: 1M, Resistor_SMD:R_0805_2012Metric
- added D1: SMF9.0CA, Diode_SMD:D_SOD-123, F.Cu at (148.1, 90.5)
- added J3: USB_C_Receptacle_USB2.0, Connector_USB:USB_C_Receptacle_HRO_TYPE-C-31-M-12, F.Cu at (136.7, 88.1)
- R1, R2: value 5.1k -> 5k1; footprint Resistor_SMD:R_0603_1608Metric -> Resistor_SMD:R_0402_1005Metric
- moved F1 3.78 mm to (145.7, 90.5), turned to -90 degrees
- moved R1 2.81 mm to (142.9, 91.3)
- moved R2 0.24 mm to (144.1, 91.3)
Connections:
- F1 pad 2: VCC -> VBUS
- MH1 pad 1: SHIELD -> GND
- MH2 pad 1: SHIELD -> GND
- R1 pad 1: Net-(J1-Pad10) -> /CC1
- R2 pad 1: Net-(J1-Pad4) -> /CC2
Routing:
- net SHIELD: track 56.6 -> 0.00 mm
- net VCC: track 27.6 -> 0.00 mm
- net VBUS: track 0.00 -> 14.5 mm, vias 0 -> 2
- net Net-(J1-Pad10): track 13.7 -> 0.00 mm, vias 2 -> 0
- net /CC2: track 0.00 -> 13.1 mm, vias 0 -> 2
- net GND: track 19.1 -> 6.94 mm, vias 7 -> 2
- net Net-(J1-Pad4): track 8.72 -> 0.00 mm, vias 2 -> 0
- net /CC1: track 0.00 -> 7.69 mm, vias 0 -> 2
- net +5V: track 25.3 -> 29.8 mm, vias 0 -> 2
- net D+: track 17.7 -> 17.1 mm
